File: Docs/PCBs/Car_0.sch (EAGLE design)
At the start: 17 parts, among them IC1 L298, U1 RASPI3_GPIO, U2 NCP59301DS50R4G

Commit message: Comments updated
Other:
- moved on the sheet: C1, C2, D1, D2, D3, D4, D5, D6, D7, D8, IC1, R1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
