File: Docs/PCBs/host_0.sch (EAGLE design)
At the start: 13 parts, among them IC1 MCP23S17SS, IC3 LM2901DSO-14, IC4 LM2901DSO-14, IC5 LM2901DSO-14, IC6 LM2901DSO-14, U1 RASPI3_GPIO

Commit message: Comments updated
Parts:
- R5: value 10k -> 4.7k
Other:
- note added: "Author: Minghao Cheng Pacman"
- moved on the sheet: C1, IC1, IC3, IC4, IC5, IC6, JP2, JP3, R1, R2, R5, R6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
