File: Docs/PCBs/host_1.sch (EAGLE design)
At the start: 30 parts, among them IC2 MCP23S17SS, Q1 BCW60SMD, Q10 BCW60SMD, Q11 BCW60SMD, Q12 BCW60SMD, Q13 BCX71SMD, Q14 BCX71SMD, Q15 BCX71SMD, Q16 BCX71SMD, Q2 BCW60SMD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

Commit message: Comments updated
Other:
- note added: "Author: Minghao Cheng Pacman"
Changed lines of the file:
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@@
 <layers>
 <layer number="1" name="Top" color="4" fill="1" visible="no" active="no"/>
+<layer number="2" name="Route2" color="1" fill="3" visible="no" active="no"/>
+<layer number="3" name="Route3" color="4" fill="3" visible="no" active="no"/>
+<layer number="4" name="Route4" color="1" fill="4" visible="no" active="no"/>
+<layer number="5" name="Route5" color="4" fill="4" visible="no" active="no"/>
+<layer number="6" name="Route6" color="1" fill="8" visible="no" active="no"/>
+<layer number="7" name="Route7" color="4" fill="8" visible="no" active="no"/>
+<layer number="8" name="Route8" color="1" fill="2" visible="no" active="no"/>
+<layer number="9" name="Route9" color="4" fill="2" visible="no" active="no"/>
+<layer number="10" name="Route10" color="1" fill="7" visible="no" active="no"/>
+<layer number="11" name="Route11" color="4" fill="7" visible="no" active="no"/>
+<layer number="12" name="Route12" color="1" fill="5" visible="no" active="no"/>
+<layer number="13" name="Route13" color="4" fill="5" visible="no" active="no"/>
+<layer number="14" name="Route14" color="1" fill="6" visible="no" active="no"/>
+<layer number="15" name="Route15" color="4" fill="6" visible="no" active="no"/>
 <layer number="16" name="Bottom" color="1" fill="1" visible="no" active="no"/>
 <layer number="17" name="Pads" color="2" fill="1" visible="no" active="no"/>
@@
 <part name="P+2" library="supply1" library_urn="urn:adsk.eagle:library:371" deviceset="VCC" device=""/>
 <part name="P+4" library="supply1" library_urn="urn:adsk.eagle:library:371" deviceset="VCC" device=""/>
+<part name="FRAME1" library="frames" deviceset="FRAME_C_L" device=""/>
 </parts>
 <sheets>
 <sheet>
 <plain>
+<text x="329.438" y="-204.978" size="2.54" layer="94">Author:     Minghao Cheng
+Pacman</text>
 </plain>
 <instances>
@@
 <instance part="P+4" gate="VCC" x="157.48" y="-12.7" smashed="yes" rot="MR270">
 <attribute name="VALUE" x="160.02" y="-10.16" size="1.778" layer="96" rot="MR0"/>
+</instance>
+<instance part="FRAME1" gate="G$1" x="-124.46" y="-231.14" smashed="yes"/>
+<instance part="FRAME1" gate="G$2" x="327.66" y="-231.14" smashed="yes">
+<attribute name="LAST_DATE_TIME" x="340.36" y="-229.87" size="2.54" layer="94"/>
+<attribute name="SHEET" x="414.02" y="-229.87" size="2.54" layer="94"/>
+<attribute name="DRAWING_NAME" x="345.44" y="-212.09" size="2.54" layer="94"/>
 </instance>
 </instances>
@@
 </drawing>
 <compatibility>
+<note version="6.3" minversion="6.2.2" severity="warning">
+Since Version 6.2.2 text objects can contain more than one line,
+which will not be processed correctly with this version.
+</note>
 <note version="8.2" severity="warning">
 Since Version 8.2, EAGLE supports online libraries. The ids
